Commit message: Imported upstream version '4.17.1' of 'upstream'

File: tiago_description/ros2_control/ros2_control.urdf.xacro (robot description, xacro)
@@ -17,5 +17,4 @@
   <xacro:include filename="$(find tiago_description)/urdf/head/head.ros2_control.xacro" />
   <xacro:include filename="$(find ${base_type}_description)/urdf/wheels/wheel.ros2_control.xacro" />
-  <xacro:include filename="$(find ${base_type}_description)/urdf/sensors/sensors.ros2_control.xacro"/>
   <xacro:include filename="${eye_hand_calibration_dir}/eye_hand_calibration.urdf.xacro" />
   <!-- Arm, Wrist, FT, EE -->
@@ -56,6 +55,4 @@
         <xacro:if value="${use_sim_time}">
           <plugin>gazebo_ros2_control/GazeboSystem</plugin>
-        <!-- IMU sensor (only in simulation)-->
-        <xacro:ros2_control_imu name="base_imu_sensor"/>
         </xacro:if>
         <xacro:unless value="${use_sim_time}">
@@ -73,8 +70,4 @@
         <xacro:ros2_control_wheel side="rear_right" />
         <xacro:ros2_control_wheel side="rear_left" />
-      </xacro:if>
-      <!-- IMU -->
-      <xacro:if value="${use_sim_time}">
-        <xacro:ros2_control_imu name="base_imu_sensor"/>
       </xacro:if>
       <!-- Torso -->

File: tiago_description/urdf/sensors/openni.gazebo.xacro (robot description, xacro)
@@ -17,5 +17,5 @@
   <!-- MACRO DEFINITION-->
   <xacro:macro name="openni_camera_gazebo_v0" params="name">
-    <gazebo reference="${name}_rgb_frame">
+    <gazebo reference="${name}_color_frame">
       <sensor type="depth" name="${name}_frame_sensor">
         <always_on>true</always_on>
@@ -46,9 +46,9 @@
             <remapping>${name}/image_raw:=${name}/rgb/image_raw</remapping>
             <remapping>${name}/camera_info:=${name}/rgb/camera_info</remapping>
-            <remapping>${name}/depth/image_raw:=${name}/depth_registered/image_raw</remapping>
-            <remapping>${name}/depth/camera_info:=${name}/depth_registered/camera_info</remapping>
-            <remapping>${name}/points:=${name}/depth_registered/points</remapping>
+            <remapping>${name}/depth/image_raw:=${name}/depth/image_raw</remapping>
+            <remapping>${name}/depth/camera_info:=${name}/depth/camera_info</remapping>
+            <remapping>${name}/points:=${name}/depth/points</remapping>
           </ros>
-          <frame_name>${name}_rgb_optical_frame</frame_name>
+          <frame_name>${name}_color_optical_frame</frame_name>
           <min_depth>0.3</min_depth>
           <max_depth>8.0</max_depth>

File: tiago_description/urdf/sensors/orbbec_astra.urdf.xacro (robot description, xacro)
@@ -81,5 +81,5 @@
     <joint name="${name}_depth_joint" type="fixed">
       <xacro:camera_baseline_constants camera_model="${camera_model}" />
-      <parent link="${name}_rgb_frame" />
+      <parent link="${name}_color_frame" />
       <child link="${name}_depth_frame"/>
     </joint>
@@ -104,10 +104,10 @@
     </link>
     <!-- frames of the rgb sensor -->
-    <joint name="${name}_rgb_joint" type="fixed">
+    <joint name="${name}_color_joint" type="fixed">
       <origin xyz="0.0 0.022 0.0" rpy="0 0 0" />
       <parent link="${name}_orbbec_aux_joint_frame" />
-      <child link="${name}_rgb_frame"/>
+      <child link="${name}_color_frame"/>
     </joint>
-    <link name="${name}_rgb_frame">
+    <link name="${name}_color_frame">
       <inertial>
         <origin xyz="0 0 0" rpy="0 0 0"/>
@@ -116,10 +116,10 @@
       </inertial>
     </link>
-    <joint name="${name}_rgb_optical_joint" type="fixed">
+    <joint name="${name}_color_optical_joint" type="fixed">
       <origin xyz="0 0 0" rpy="${-90.0 * deg_to_rad} 0.0 ${-90.0 * deg_to_rad}" />
-      <parent link="${name}_rgb_frame" />
-      <child link="${name}_rgb_optical_frame"/>
+      <parent link="${name}_color_frame" />
+      <child link="${name}_color_optical_frame"/>
     </joint>
-    <link name="${name}_rgb_optical_frame">
+    <link name="${name}_color_optical_frame">
       <inertial>
         <origin xyz="0 0 0" rpy="0 0 0"/>

File: tiago_description/urdf/sensors/xtion_pro_live.urdf.xacro (robot description, xacro)
@@ -86,10 +86,10 @@
     </link>
     <!-- frames of the rgb sensor -->
-    <joint name="${name}_rgb_joint" type="fixed">
+    <joint name="${name}_color_joint" type="fixed">
       <origin xyz="0.0 0.022 0.0" rpy="0 0 0" />
       <parent link="${name}_link" />
-      <child link="${name}_rgb_frame"/>
+      <child link="${name}_color_frame"/>
     </joint>
-    <link name="${name}_rgb_frame">
+    <link name="${name}_color_frame">
       <inertial>
         <origin xyz="0 0 0" rpy="0 0 0"/>
@@ -98,10 +98,10 @@
       </inertial>
     </link>
-    <joint name="${name}_rgb_optical_joint" type="fixed">
+    <joint name="${name}_color_optical_joint" type="fixed">
       <origin xyz="0 0 0" rpy="${-90.0 * deg_to_rad} 0.0 ${-90.0 * deg_to_rad}" />
-      <parent link="${name}_rgb_frame" />
-      <child link="${name}_rgb_optical_frame"/>
+      <parent link="${name}_color_frame" />
+      <child link="${name}_color_optical_frame"/>
     </joint>
-    <link name="${name}_rgb_optical_frame">
+    <link name="${name}_color_optical_frame">
       <inertial>
         <origin xyz="0 0 0" rpy="0 0 0"/>
