Commit message: Imported upstream version '4.6.0' of 'upstream'

File: tiago_description/robots/tiago.urdf.xacro (robot description, xacro)
@@ -140,5 +140,12 @@
   </xacro:if>
   <!-- Torso -->
-  <xacro:tiago_torso name="torso" parent="base_link"/>
+  <xacro:tiago_torso name="torso" parent="base_link">
+    <xacro:if value="${base_type == 'pmb2'}">
+      <origin rpy="0 0 0" xyz="-0.062 0.0 0.193" />
+    </xacro:if>
+    <xacro:if value="${base_type == 'omni_base'}">
+      <origin rpy="0 0 0" xyz="-0.062 0.0 0.215" />
+    </xacro:if>
+  </xacro:tiago_torso>
   <!-- Arm, FT, EE -->
   <xacro:if value="${has_arm}">

Commit message: Imported upstream version '4.14.0' of 'upstream'

File: tiago_description/robots/tiago.urdf.xacro (robot description, xacro)
@@ -44,6 +44,6 @@
   <xacro:arg name="no_safety_eps" default="false"/>
   <!-- Calibration -->
-  <xacro:arg name="description_calibration_dir" default="$(find tiago_description)/urdf/calibration"/>
-  <xacro:arg name="extrinsic_calibration_dir" default="$(find tiago_description)/urdf/calibration"/>
+  <xacro:arg name="eye_hand_calibration_dir" default="$(find tiago_description)/urdf/calibration"/>
+  <xacro:arg name="camera_extrinsic_calibration_dir" default="$(find tiago_description)/urdf/calibration"/>
   <!-- Execution env config -->
   <xacro:arg name="use_sim_time" default="false"/>
@@ -98,6 +98,6 @@
   <xacro:property name="arm_yaw" default="-90" />
   <!-- Calibration -->
-  <xacro:property name="description_calibration_dir" value="$(arg description_calibration_dir)"/>
-  <xacro:property name="extrinsic_calibration_dir" value="$(arg extrinsic_calibration_dir)"/>
+  <xacro:property name="eye_hand_calibration_dir" value="$(arg eye_hand_calibration_dir)"/>
+  <xacro:property name="camera_extrinsic_calibration_dir" value="$(arg camera_extrinsic_calibration_dir)"/>
   <!-- Execution env configuration -->
   <xacro:property name="use_sim_time" default="$(arg use_sim_time)"/>

File: tiago_description/ros2_control/ros2_control.urdf.xacro (robot description, xacro)
@@ -18,5 +18,5 @@
   <xacro:include filename="$(find ${base_type}_description)/urdf/wheels/wheel.ros2_control.xacro" />
   <xacro:include filename="$(find ${base_type}_description)/urdf/sensors/sensors.ros2_control.xacro"/>
-  <xacro:include filename="${description_calibration_dir}/calibration_constants.urdf.xacro" />
+  <xacro:include filename="${eye_hand_calibration_dir}/eye_hand_calibration.urdf.xacro" />
   <!-- Arm, Wrist, FT, EE -->
   <xacro:if value="${has_arm}">

File: tiago_description/urdf/end_effector/end_effector.urdf.xacro (robot description, xacro)
@@ -31,5 +31,5 @@
     <xacro:if value="${end_effector == 'pal-gripper'}">
       <xacro:pal_gripper parent="${parent}" name="${name}">
-        <origin xyz="0.01 0 0" rpy="${90*deg_to_rad} ${90*deg_to_rad} ${-90*deg_to_rad}"/>
+        <origin xyz="0 0 0" rpy="${90*deg_to_rad} ${90*deg_to_rad} ${-90*deg_to_rad}"/>
       </xacro:pal_gripper>
     </xacro:if>
@@ -37,5 +37,5 @@
     <xacro:if value="${end_effector == 'robotiq-2f-85'}">
       <xacro:robotiq_85_gripper prefix="${name}_" parent="${parent}">
-        <origin xyz="0.01 0 0" rpy="${90*deg_to_rad} ${0*deg_to_rad} ${90*deg_to_rad}"/>
+        <origin xyz="0 0 0" rpy="${90*deg_to_rad} ${0*deg_to_rad} ${90*deg_to_rad}"/>
       </xacro:robotiq_85_gripper>
     </xacro:if>
@@ -43,5 +43,5 @@
     <xacro:if value="${end_effector == 'robotiq-2f-140'}">
       <xacro:robotiq_140_gripper prefix="${name}_" parent="${parent}">
-        <origin xyz="0.01 0 0" rpy="${90*deg_to_rad} ${0*deg_to_rad} ${90*deg_to_rad}"/>
+        <origin xyz="0 0 0" rpy="${90*deg_to_rad} ${0*deg_to_rad} ${90*deg_to_rad}"/>
       </xacro:robotiq_140_gripper>
     </xacro:if>
@@ -57,17 +57,4 @@
       </joint>
       <link name="${name}_safety_box">
-        <inertial>
-          <origin xyz="0 0 0" rpy="0 0 0"/>
-          <mass value="0.0001" />
-          <inertia ixx="0.0001" ixy="0" ixz="0" iyy="0.0001" iyz="0" izz="0.0001" />
-        </inertial>
-        <!--
-      <visual>
-        <origin xyz="0 0 0" rpy="0 0 0" />
-        <geometry>
-          <box size="0.2 0.115 0.18" />
-        </geometry>
-      </visual>
-      -->
         <collision>
           <origin xyz="0 0 0" rpy="0 0 0" />

File: tiago_description/urdf/head/head.urdf.xacro (robot description, xacro)
@@ -27,5 +27,5 @@
   <xacro:include filename="$(find tiago_description)/urdf/sensors/xtion_pro_live.urdf.xacro" />
   <xacro:include filename="$(find tiago_description)/urdf/sensors/orbbec_astra.urdf.xacro" />
-  <xacro:include filename="$(arg description_calibration_dir)/calibration_constants.urdf.xacro" />
+  <xacro:include filename="$(arg eye_hand_calibration_dir)/eye_hand_calibration.urdf.xacro" />
   <!-- MACRO DEFINITION-->
   <!-- head_1 (pan) -->
@@ -109,5 +109,5 @@
     <!-- Asus Xtion-->
     <xacro:if value="${camera_model == 'asus-xtion'}">
-      <xacro:xtion_pro_live name="head_front_camera" parent="${name}_2_link" camera_model="${camera_model}" extrinsic_calibration_dir="${extrinsic_calibration_dir}">
+      <xacro:xtion_pro_live name="head_front_camera" parent="${name}_2_link" camera_model="${camera_model}" camera_extrinsic_calibration_dir="${camera_extrinsic_calibration_dir}">
         <origin xyz="${camera_position_x} ${camera_position_y} ${camera_position_z}" rpy="${camera_orientation_r} ${camera_orientation_p} ${camera_orientation_y}" />
         <!-- optical origin -->
@@ -117,5 +117,5 @@
     <!-- Orbecc Astra-->
     <xacro:if value="${camera_model in ['orbbec-astra', 'orbbec-astra-pro']}">
-      <xacro:orbbec_astra name="head_front_camera" parent="${name}_2_link" camera_model="${camera_model}" extrinsic_calibration_dir="${extrinsic_calibration_dir}">
+      <xacro:orbbec_astra name="head_front_camera" parent="${name}_2_link" camera_model="${camera_model}" camera_extrinsic_calibration_dir="${camera_extrinsic_calibration_dir}">
         <origin xyz="${camera_position_x} ${camera_position_y} ${camera_position_z}" rpy="${camera_orientation_r} ${camera_orientation_p} ${camera_orientation_y}" />
         <!-- optical origin -->

File: tiago_description/urdf/sensors/orbbec_astra.urdf.xacro (robot description, xacro)
@@ -16,7 +16,7 @@
   <!-- INCLUDES -->
   <xacro:include filename="$(find tiago_description)/urdf/sensors/openni.gazebo.xacro" />
-  <xacro:include filename="${extrinsic_calibration_dir}/extrinsic_camera_calibration_constants.urdf.xacro" />
+  <xacro:include filename="${camera_extrinsic_calibration_dir}/camera_extrinsic_calibration.urdf.xacro" />
   <!-- MACRO DEFINITION-->
-  <xacro:macro name="orbbec_astra" params="name parent camera_model *origin *optical_origin extrinsic_calibration_dir">
+  <xacro:macro name="orbbec_astra" params="name parent camera_model *origin *optical_origin camera_extrinsic_calibration_dir">
     <!-- frames in the center of the camera -->
     <joint name="${name}_joint" type="fixed">

File: tiago_description/urdf/sensors/xtion_pro_live.urdf.xacro (robot description, xacro)
@@ -15,7 +15,7 @@
   <!-- INCLUDES -->
   <xacro:include filename="$(find tiago_description)/urdf/sensors/openni.gazebo.xacro" />
-  <xacro:include filename="${extrinsic_calibration_dir}/extrinsic_camera_calibration_constants.urdf.xacro" />
+  <xacro:include filename="${camera_extrinsic_calibration_dir}/camera_extrinsic_calibration.urdf.xacro" />
   <!-- MACRO DEFINITION-->
-  <xacro:macro name="xtion_pro_live" params="name parent camera_model *origin *optical_origin extrinsic_calibration_dir">
+  <xacro:macro name="xtion_pro_live" params="name parent camera_model *origin *optical_origin camera_extrinsic_calibration_dir">
     <!-- frames in the center of the camera -->
     <joint name="${name}_joint" type="fixed">

Commit message: Imported upstream version '4.22.0' of 'upstream'

File: tiago_description/robots/tiago.urdf.xacro (robot description, xacro)
@@ -140,5 +140,5 @@
   </xacro:if>
   <!-- Torso -->
-  <xacro:tiago_torso name="torso" parent="base_link">
+  <xacro:tiago_torso name="torso" parent="base_link" has_screen="${has_screen}">
     <xacro:if value="${base_type == 'pmb2'}">
       <origin rpy="0 0 0" xyz="-0.062 0.0 0.193" />

File: tiago_description/urdf/torso/torso.urdf.xacro (robot description, xacro)
@@ -19,5 +19,5 @@
   <xacro:include filename="$(find pal_urdf_utils)/urdf/deg_to_rad.urdf.xacro" />
   <!-- MACRO DEFINITION-->
-  <xacro:macro name="tiago_torso" params="name parent *origin">
+  <xacro:macro name="tiago_torso" params="name parent *origin has_screen">
     <!-- Bottom fixed part of column -->
     <link name="${name}_fixed_link">
@@ -70,5 +70,5 @@
         <origin rpy="0 0 0" xyz="0 0 0.275" />
         <geometry>
-          <box size="0.23 0.23 0.55"/>
+          <box size="0.232 0.265 0.45"/>
         </geometry>
         <material name="DarkGrey"/>
@@ -119,4 +119,20 @@
         <material name="LightGrey"/>
       </collision>
+    <xacro:if value="$(arg has_screen)">
+      <visual>
+        <origin rpy="0 0 -1.57" xyz="-0.01 0.125 -0.27" />
+        <geometry>
+          <mesh filename="package://tiago_description/meshes/torso/tiago_screen.stl" scale="1 1 1"/>
+        </geometry>
+        <material name="White"/>
+      </visual>
+      <collision>
+        <origin rpy="0 0 -1.57" xyz="-0.01 0.125 -0.27" />
+        <geometry>
+          <mesh filename="package://tiago_description/meshes/torso/tiago_screen_collision.stl" scale="1 1 1"/>
+        </geometry>
+        <material name="LightGrey"/>
+      </collision>
+    </xacro:if>
     </link>
     <joint name="${name}_lift_joint" type="prismatic">
