Commit message: Imported upstream version '4.24.1' of 'upstream'

File: tiago_description/urdf/arm/arm.urdf.xacro (robot description, xacro)
@@ -43,5 +43,5 @@
         <origin xyz="0.061191 -0.022397 ${reflect * -0.012835}" rpy="0.00000 0.00000 0.00000"/>
         <mass value="1.563428"/>
-        <inertia ixx="0.002471" ixy="${reflect * -0.001809}" ixz="-0.001202" iyy="0.006132" iyz="${reflect * 0.000494}" izz="0.006704"/>
+        <inertia ixx="0.002471" ixy="${-reflect * -0.001809}" ixz="-0.001202" iyy="0.006132" iyz="${reflect * 0.000494}" izz="0.006704"/>
       </inertial>
       <!-- M90 module -->

File: tiago_description/urdf/torso/torso.urdf.xacro (robot description, xacro)
@@ -136,4 +136,12 @@
     </xacro:if>
     </link>
+    <!-- TODO: set lower limit back to 0 when moving to Gazebo Harmonic or ROS 2 Jazzy -->
+    <!-- See https://github.com/gazebosim/gz-sim/issues/1684 for more information -->
+    <xacro:if value="${gazebo_version == 'classic'}">
+      <xacro:property name="torso_lower_limit" value="0.0"/>
+    </xacro:if>
+    <xacro:if value="${gazebo_version == 'gazebo'}">
+      <xacro:property name="torso_lower_limit" value="-1e-3"/>
+    </xacro:if>
     <joint name="${name}_lift_joint" type="prismatic">
       <origin rpy="0.0 0.0 0.0" xyz="0.0 0.0 0.597" />
@@ -141,5 +149,5 @@
       <child link="${name}_lift_link" />
       <axis xyz="0 0 1" />
-      <limit effort="2000" lower="0" upper="0.35" velocity="${torso_max_vel}" />
+      <limit effort="2000" lower="${torso_lower_limit}" upper="0.35" velocity="${torso_max_vel}" />
       <calibration rising="0.0" />
       <dynamics damping="1000" />
